File: wifi_pants.sch (KiCad schematic (older format))
At the start: 24 parts, among them P1 CONN_02X20, P2 CONN_01X10, U1 ESP-12E

Commit message: start adding boost converter
Parts:
- removed JP3: FORCE_HOLD, wifi_pants:GS2, symbol Jumper_NO_Small
- removed JP5: WP_DISABLE, wifi_pants:GS2, symbol Jumper_NO_Small
- added C? (x3): 10uF, Capacitors_SMD:C_0805_HandSoldering, symbol C
- added C?: 100pF, Capacitors_SMD:C_0805_HandSoldering, symbol C
- added L?: INDUCTOR, symbol INDUCTOR
- added P?: CONN_01X02, symbol CONN_01X02
- added R?: 150, Resistors_SMD:R_0603_HandSoldering, symbol R
- added R?: 20K, Resistors_SMD:R_0603_HandSoldering, symbol R
- added R?: 768K, Resistors_SMD:R_0603_HandSoldering, symbol R
- added R?: 243K, Resistors_SMD:R_0603_HandSoldering, symbol R
- added U?: TPS61252, Housings_DFN_QFN:DFN-8-1EP_2x2mm_Pitch0.5mm, symbol TPS61252
- R1, R6: value 150-DNP -> 150
Connections:
- net +3V3: no longer R1.2, U1.12 (GPIO10)
- net GND: now also C?.2, P?.2 (P2), R?.2, R?.2, U?.1 (GND), U?.9 (GND)
- net AUDIO_L: now reaches P2.8 (P8)
- net AUDIO_L: now also C5.1; no longer C4.1
- net AUDIO_R: now reaches P2.9 (P9)
- net AUDIO_R: now also C4.1; no longer C5.1
- new net: C?.1, C?.2, R?.1, U?.2 (VOUT)
- new net: C?.1, C?.2, R?.1, R?.2, U?.3 (FB)
- new net: R?.1, U?.4 (ILIM)
- new net: L?.2, U?.7 (SW)
- new net: C?.1, L?.1, P?.1 (P1), R?.1, U?.8 (VIN)
- new net /WP: R1.2, U1.12 (GPIO10)
- new net PS_EN: R?.2, U?.6 (EN)
- no-connect marks 32 -> 33
Other:
- note removed: "FTDI 6-pin"
- note removed: "For 4-bit SDIO, populate the\nSD_D2 and SD_D3 resistors\nand cut JP5. Use with ESP-12F\nmodule with removed flash or\nproposed SPI flash sleep mode"
- note removed: "Solder JP3 in ICT\nafter disabling\nQSPI mode on\nmodule\n"
- moved on the sheet: C2, C3, C4, C5, R10, R7, R8, R9
